Commit message: Alaa - modifying errors made by git and merging

File: catkin/src/cwru_376_student/cwru_urdf/abby_w_arm_urdf_rviz_only.xacro (robot description, xacro)
@@ -723,15 +723,8 @@
   <joint name="kinect_joint" type="fixed">
       <axis xyz="0 1 0" />
-<<<<<<< HEAD
-      <origin xyz="0.45 0 1.65" rpy="0 0.92 0"/>
-=======
       <origin xyz="0.55 0.03 1.585" rpy="0.06 0.95 0"/>
->>>>>>> upstream/master
       <parent link="base_link"/>
       <child link="kinect_link"/>
   </joint>
-<<<<<<< HEAD
-=======
->>>>>>> upstream/master
 <gazebo>
   <plugin name="differential_drive_controller" filename="libgazebo_ros_diff_drive.so">
